File: EnvelopeCrusher/ MicroController.kicad_sch (KiCad schematic)
At the start: 11 parts

Commit message: Add routing
Parts:
- added JP? (x2): SolderJumper_2_Bridged, Jumper:SolderJumper-2_P1.3mm_Bridged_Pad1.0x1.5mm, symbol Jumper:SolderJumper_2_Bridged
- added U?: MCP603-xCH, Package_TO_SOT_SMD:SOT-23-6, symbol Amplifier_Operational:MCP603-xCH
Connections:
- net +3V3: now also U?.6 (V+)
- net GND: now also U?.2 (V-), U?.5 (~{CS})
- net PA4: now reaches U?.10 (PA4)
- net PA4: now also JP?.1 (A)
- net PA5: now reaches U?.11 (PA5)
- net PA5: now also JP?.1 (A)
- net PA0: now reaches U?.6 (PA0)
- net PA0: now also U?.1, U?.4 (-)
- new net EnvelopeGen1: JP?.2 (B)
- new net EnvelopeGen2: JP?.2 (B)
- new net PEAK_IN1: U?.3 (+)
Other:
- moved on the sheet: C?, J?, JP?, SW?

Commit message: updated
Parts:
- removed JP? (x2): SolderJumper_2_Bridged, Jumper:SolderJumper-2_P1.3mm_Bridged_Pad1.0x1.5mm, symbol Jumper:SolderJumper_2_Bridged
- added D?: LED, symbol Device:LED
- added J?: Conn_01x02, Connector_PinHeader_2.54mm:PinHeader_1x02_P2.54mm_Vertical, symbol Connector_Generic:Conn_01x02
- added J?: Conn_01x04, symbol Connector_Generic:Conn_01x04
- added JP? (x4): SolderJumper_2_Bridged, symbol Jumper:SolderJumper_2_Bridged
- added R? (x2): 10K, Resistor_SMD:R_0805_2012Metric_Pad1.20x1.40mm_HandSolder, symbol Device:R
- added R?: 2K2, Resistor_SMD:R_0805_2012Metric_Pad1.20x1.40mm_HandSolder, symbol Device:R
- added SW?: RotaryEncoder_Switch, Rotary_Encoder:RotaryEncoder_Alps_EC11E-Switch_Vertical_H20mm, symbol Device:RotaryEncoder_Switch
Connections:
- net +3V3: now also JP?.2 (B), R?.1, R?.1
- net GND: now also D?.1 (K), J?.1 (Pin_1), JP?.2 (B), SW?.C, SW?.S2
- net PA6: now reaches U?.12 (PA6)
- net RELAY_SIGNAL: now reaches U?.13 (PA7)
- net PA8: now reaches U?.18 (PA8)
- net PA8: now also R?.1
- net PA9: now reaches U?.19 (PA9)
- net PA9: now also JP?.2 (B)
- net PA10: now reaches U?.20 (PA10)
- net PA10: now also JP?.2 (B)
- net PA15: now reaches U?.25 (PA15)
- net PA15: now also R?.2, SW?.B
- net PB3: now reaches U?.26 (PB3)
- net PB3: now also R?.2, SW?.A
- net PB4: now reaches U?.27 (PB4)
- net PB4: now also SW?.S1
- net PA2: now reaches U?.8 (PA2)
- net PA3: now reaches U?.9 (PA3)
- net PA3: now also J?.2 (Pin_2)
- new net: J?.3 (Pin_3), JP?.1 (A)
- new net: J?.4 (Pin_4), JP?.1 (A)
- new net: J?.2 (Pin_2), JP?.1 (A)
- new net: J?.1 (Pin_1), JP?.1 (A)
- new net: D?.2 (A), R?.2
Other:
- added sheet ENV_CLK_MIX (ENV_CLK_MIX.kicad_sch)
- note added: "ADC1_IN5"
- note added: "DAC1_OUT1 (TIM6)"
- note added: "DAC1_OUT2 (TIM7)"
- note added: "ENCODER MODE (Pin A)"
- note added: "ENCODER MODE (Pin B)"
- note added: "EXTI4 (Pin S1)"
- note added: "FOOTSWITCH"
- note added: "GPIO OUTPUT (LED)"
- note added: "GPIO OUTPUT (Relay)"
- note added: "I2C_SCL"
- note added: "I2C_SDA"
- note added: "TIM15_CH1 (PWM)"
- note added: "TIM16_CH1 (PWM)"
- moved on the sheet: C?, J?, JP?, SW?, U?

Commit message: Completed Schematic
Parts:
- added C16: 100nF, Capacitor_SMD:C_0805_2012Metric_Pad1.18x1.45mm_HandSolder, symbol Device:C
- added C21: 1uF, Capacitor_SMD:C_0805_2012Metric_Pad1.18x1.45mm_HandSolder, symbol Device:C
- added C55: 10uF, Capacitor_SMD:C_0805_2012Metric_Pad1.18x1.45mm_HandSolder, symbol Device:C
- added JP11: SolderJumper_2_Bridged, symbol Jumper:SolderJumper_2_Bridged
- added R12: 100R, Capacitor_SMD:C_0805_2012Metric_Pad1.18x1.45mm_HandSolder, symbol Device:R
- added TP1, TP10, TP11, TP12, TP13, TP14, TP15, TP16, TP17, TP18, TP19, TP2, TP20, TP21, TP22, TP23, TP24, TP25, TP3, TP4, TP5, TP6, TP7, TP8, TP9: TestPoint, TestPoint:TestPoint_Pad_1.0x1.0mm, symbol Connector:TestPoint
- added U16: SE82XX-33, Package_TO_SOT_SMD:SOT-223-3_TabPin2, symbol Regulator_Linear:AP1117-33
- gave numbers to parts that had none: 23
Connections:
- net +3V3: now also U7.5 (VDDA), C55.1, U16.2 (VO)
- net GND: now also C16.2, C21.2, C55.2, U16.1 (GND)
- net PA0: now also C16.1, R12.2, TP10.1; no longer U2.1, U2.4 (-)
- net PA10: now also TP20.1
- net PA15: now also TP25.1
- net PA2: now also TP12.1
- net PA3: now also TP13.1
- net PA4: now also TP14.1
- net PA5: now also TP15.1
- net PA6: now also TP16.1
- net PA8: now also TP18.1
- net PA9: now also TP19.1
- net PB3: now also TP5.1
- net PB4: now also TP6.1
- net RELAY_SIGNAL: now also JP11.1 (A); no longer U7.13 (PA7)
- net SWCLK: now also TP24.1
- net SWDIO: now also TP23.1
- net PB0: now reaches U7.14 (PB0)
- net PB0: now also TP3.1
- net PB1: now reaches U7.15 (PB1)
- net PB1: now also TP4.1
- net PC14: now reaches U7.2 (PC14)
- net PC14: now also TP1.1
- net PA11: now reaches U7.21 (PA11)
- net PA11: now also TP21.1
- net PA12: now reaches U7.22 (PA12)
- net PA12: now also TP22.1
- net PB5: now reaches U7.28 (PB5)
- net PB5: now also TP7.1
- net PB6: now reaches U7.29 (PB6)
- net PB6: now also TP8.1
- net PC15: now reaches U7.3 (PC15)
- net PC15: now also TP2.1
- net PB7: now reaches U7.30 (PB7)
- net PB7: now also TP9.1
- net PA1: now reaches U7.7 (PA1)
- net PA1: now also TP11.1
- new net: R12.1, U2.1, U2.4 (-)
- new net +9V: C21.1, U16.3 (VI)
- new net PA7: JP11.2 (B), TP17.1, U7.13 (PA7)
Other:
- note added: "100nF close to each VDD"
- note added: "10nF close to VDDA"
- note added: "NC"
- moved on the sheet: C5, C6, D1, J1, J2, J3, JP3, JP4, JP5, JP6, R1, R2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

Commit message: updated schematic
- Added values and comments to state-variable filter block
- Updated footprints
- Changed Dual Op Amp: TL072 to AM358
Parts:
- D1: footprint (none) -> LED_SMD:LED_0805_2012Metric_Pad1.15x1.40mm_HandSolder
- J3: footprint (none) -> Connector_PinHeader_2.54mm:PinHeader_1x04_P2.54mm_Vertical
- JP1: footprint (none) -> Jumper:SolderJumper-2_P1.3mm_Open_Pad1.0x1.5mm
- JP11, JP2, JP3, JP4, JP5, JP6: footprint (none) -> Jumper:SolderJumper-2_P1.3mm_Bridged_Pad1.0x1.5mm
- R12: footprint Capacitor_SMD:C_0805_2012Metric_Pad1.18x1.45mm_HandSolder -> Resistor_SMD:R_0805_2012Metric_Pad1.20x1.40mm_HandSolder
Other:
- note added: "10-Pin ARM Programming Header"
- note added: "Decoupling Capacitors"
- note added: "Dedicated Voltage Regulator"
- note added: "Envelope/Clock Mixer Output Stage"
- note added: "FOOTSWITCH (EXTI3)"
- note added: "Microcontroller"
- note added: "OLED Display Connector"
- note added: "Peak Detector Input Buffer for ADC"
- note added: "Rotary Encoder"
- note added: "Signal Path Footswitch Connector"
- note added: "Signal Path LED"
- note added: "Signal Path Relay"
- note added: "Testpoints"
- note removed: "FOOTSWITCH"
- moved on the sheet: C1, C16, C2, C21, C3, C4, C5, C55, C6, D1, J1, J2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

Commit message: started layout
Parts:
- removed SW3: SW_SPST, symbol Switch:SW_SPST
- added JP12: SolderJumper_2_Open, Jumper:SolderJumper-2_P1.3mm_Open_Pad1.0x1.5mm, symbol Jumper:SolderJumper_2_Open
- J3: footprint Connector_PinHeader_2.54mm:PinHeader_1x04_P2.54mm_Vertical -> 0.96inch_OLED_SSD1306:0.96inch_OLED_SSD1306
Connections:
- net GND: now also JP12.1 (A)
- net NRST: now also JP12.2 (B)
Changed lines of the file:
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@@
     (stroke (width 0) (type default) (color 0 0 0 0))
   )
-  (wire (pts (xy 242.57 356.87) (xy 242.57 358.14))
+  (wire (pts (xy 242.57 356.87) (xy 242.57 359.41))
     (stroke (width 0) (type default) (color 0 0 0 0))
   )
@@
     (stroke (width 0) (type default) (color 0 0 0 0))
   )
-  (wire (pts (xy 242.57 368.3) (xy 242.57 369.57))
+  (wire (pts (xy 242.57 367.03) (xy 242.57 369.57))
     (stroke (width 0) (type default) (color 0 0 0 0))
   )
@@
     (pin "S1")
     (pin "S2")
-  )
-  (symbol (lib_id "Switch:SW_SPST") (at 242.57 363.22 90) (unit 1)
-    (in_bom yes) (on_board yes) (fields_autoplaced)
-    (property "Reference" "SW3" (id 0) (at 243.84 361.9499 90)
-      (effects (font (size 1.27 1.27)) (justify right))
-    )
-    (property "Value" "SW_SPST" (id 1) (at 243.84 364.4899 90)
-      (effects (font (size 1.27 1.27)) (justify right) hide)
-    )
-    (property "Footprint" "" (id 2) (at 242.57 363.22 0)
-      (effects (font (size 1.27 1.27)) hide)
-    )
-    (property "Datasheet" "~" (id 3) (at 242.57 363.22 0)
-      (effects (font (size 1.27 1.27)) hide)
-    )
-    (pin "1")
-    (pin "2")
   )
   (symbol (lib_id "Connector:TestPoint") (at 311.15 256.54 90) (unit 1)
@@
     (pin "1")
   )
+  (symbol (lib_id "Jumper:SolderJumper_2_Open") (at 242.57 363.22 90) (unit 1)
+    (in_bom yes) (on_board yes) (fields_autoplaced)
+    (property "Reference" "JP12" (id 0) (at 245.11 361.9499 90)
+      (effects (font (size 1.27 1.27)) (justify right))
+    )
+    (property "Value" "SolderJumper_2_Open" (id 1) (at 245.11 364.4899 90)
+      (effects (font (size 1.27 1.27)) (justify right) hide)
+    )
+    (property "Footprint" "Jumper:SolderJumper-2_P1.3mm_Open_Pad1.0x1.5mm" (id 2) (at 242.57 363.22 0)
+      (effects (font (size 1.27 1.27)) hide)
+    )
+    (property "Datasheet" "~" (id 3) (at 242.57 363.22 0)
+      (effects (font (size 1.27 1.27)) hide)
+    )
+    (pin "1")
+    (pin "2")
+  )
   (symbol (lib_id "Connector:TestPoint") (at 311.15 246.38 90) (unit 1)
     (in_bom yes) (on_board yes)
@@
     (property "Reference" "J3" (id 0) (at 529.59 64.77 0))
     (property "Value" "Conn_01x04" (id 1) (at 529.59 67.31 0))
-    (property "Footprint" "Connector_PinHeader_2.54mm:PinHeader_1x04_P2.54mm_Vertical" (id 2) (at 529.59 76.2 0)
-      (effects (font (size 1.27 1.27)) hide)
-    )
-    (property "Datasheet" "~" (id 3) (at 529.59 76.2 0)
-      (effects (font (size 1.27 1.27)) hide)
-    )
+    (property "Footprint" "0.96inch_OLED_SSD1306:0.96inch_OLED_SSD1306" (id 2) (at 529.59 76.2 0)
+      (effects (font (size 1.27 1.27)) hide)
+    )
+    (property "Datasheet" "http://www.lcdwiki.com/0.96inch_OLED_Module_MC096VX" (id 3) (at 529.59 76.2 0)
+      (effects (font (size 1.27 1.27)) hide)
+    )

Commit message: Updated footprints/symbol mappings
Parts:
- U16: footprint Package_TO_SOT_SMD:SOT-223-3_TabPin2 -> Package_TO_SOT_SMD:SOT-23
Changed lines of the file:
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@@
     (property "Reference" "U16" (id 0) (at 236.22 50.8 0))
     (property "Value" "SE82XX-33" (id 1) (at 236.22 53.34 0))
-    (property "Footprint" "Package_TO_SOT_SMD:SOT-223-3_TabPin2" (id 2) (at 236.22 53.34 0)
+    (property "Footprint" "Package_TO_SOT_SMD:SOT-23" (id 2) (at 236.22 53.34 0)
       (effects (font (size 1.27 1.27)) hide)
     )

Commit message: organised layout into functional blocks
Parts:
- removed C21: 1uF, Capacitor_SMD:C_0805_2012Metric_Pad1.18x1.45mm_HandSolder, symbol Device:C
- removed C55: 10uF, Capacitor_SMD:C_0805_2012Metric_Pad1.18x1.45mm_HandSolder, symbol Device:C
- removed TP1, TP10, TP11, TP12, TP13, TP14, TP15, TP16, TP17, TP18, TP19, TP2, TP20, TP21, TP22, TP23, TP24, TP25, TP3, TP4, TP5, TP6, TP7, TP8, TP9: TestPoint, TestPoint:TestPoint_Pad_1.0x1.0mm, symbol Connector:TestPoint
- removed U16: SE82XX-33, Package_TO_SOT_SMD:SOT-23, symbol Regulator_Linear:AP1117-33
- U2: renamed from U7; footprint Package_DFN_QFN:QFN-32-1EP_5x5mm_P0.5mm_EP3.45x3.45mm -> QFN-32-1EP_5x5mm_TestPoints:QFN-32-1EP_5x5mm_P0.5mm_EP3.3x3.3mm_TestPoints
- renumbered C16 to C1, C1 to C2, C2 to C3, C3 to C4, C4 to C5, C5 to C6, C6 to C7, J2 to J3, J3 to J4, JP12 to JP3, JP11 to JP4, JP3 to JP5, JP4 to JP6, JP5 to JP7, JP6 to JP8, J1 to J_FOOTSW1, R12 to R2, R2 to R3, R3 to R4, SW2 to SW3, U2 to U1
Connections:
- net SWO: no longer names the net of J3.6 (Pin_6)
- no-connect marks 2 -> 3
Other:
- note removed: "Dedicated Voltage Regulator"
- note removed: "Testpoints"
- moved on the sheet: C2, C3, C4, C5, C6, C7, J3, JP1, JP2, JP3, U2
