File: EnvelopeCrusher/EnvelopeCrusher.kicad_pcb (KiCad board)
At the start: 2 copper layers, 54.9 x 95 mm, 170 parts, among them J1 Conn_01x02, J2 Conn_02x05_Odd_Even, J3 Conn_01x04, J4 Conn_01x02, Q1 Q_NMOS_GSD, SW1 SW_SPDT, SW2 RotaryEncoder_Switch, SW4 SW_DIP_x04, SW5 SW_DPDT_x2, U1 AS358AMTR, U10 TPS60400, U11 TPS60400, U12 TPS60400, U13 TPS60400, U15 TPS60400, U16 SE82XX-33, U17 SE82XX-50, U18 SE82XX-50, U19 SE82XX-50, U2 MCP603-xCH, U20 SE82XX-50, U21 SE82XX-50, U22 SE82XX-50, U3 AS358AMTR, U4 AS358AMTR, U6 AS358AMTR, U7 STM32L432KBUx, U8 AS358AMTR, U9 TPS60400

Commit message: organised layout into functional blocks
Parts:
- removed the C21 at (97.0, 246.2)
- removed C56, C58, C60, C62, C64, C66: 1uF, Capacitor_SMD:C_0805_2012Metric_Pad1.18x1.45mm_HandSolder
- removed C57, C59, C61, C63, C65, C67: 10uF, Capacitor_SMD:C_0805_2012Metric_Pad1.18x1.45mm_HandSolder
- removed TP10, TP11, TP12, TP13, TP14, TP15, TP16, TP17, TP18, TP19, TP20, TP21, TP22, TP23, TP24, TP25, TP4, TP5, TP6, TP7, TP8, TP9: TestPoint, TestPoint:TestPoint_Pad_1.0x1.0mm
- removed U17, U18, U19, U20, U21, U22: SE82XX-50, Package_TO_SOT_SMD:SOT-223-3_TabPin2
- added C48: 10uF 20V X5R, Resistor_SMD:R_1206_3216Metric_Pad1.30x1.75mm_HandSolder, F.Cu at (-141.6, 299.7)
- added C50: 100nF, Capacitor_SMD:C_0805_2012Metric_Pad1.18x1.45mm_HandSolder, F.Cu at (-134.0, 296.5)
- added C51: 75pF, Capacitor_SMD:C_0805_2012Metric_Pad1.18x1.45mm_HandSolder, F.Cu at (-128.6, 294.8)
- added C52: 22uF 10V X5R, Resistor_SMD:R_1206_3216Metric_Pad1.30x1.75mm_HandSolder, F.Cu at (-141.6, 294.0)
- added C53: 22uF 10V X5R, Resistor_SMD:R_1206_3216Metric_Pad1.30x1.75mm_HandSolder, F.Cu at (-138.4, 294.0)
- added C54: 10uF, Capacitor_SMD:C_0805_2012Metric_Pad1.18x1.45mm_HandSolder, F.Cu at (-75.6, 286.4)
- added D10: RED, LED_SMD:LED_0805_2012Metric_Pad1.15x1.40mm_HandSolder, F.Cu at (-154.9, 293.9)
- added D11: RED, LED_SMD:LED_0805_2012Metric_Pad1.15x1.40mm_HandSolder, F.Cu at (-70.5, 286.4)
- added D9: D_Schottky, Diode_SMD:D_SOD-123F, F.Cu at (-148.1, 304.0)
- added L1: 15uH, Inductor_SMD:L_Taiyo-Yuden_NR-80xx_HandSoldering, F.Cu at (-148.0, 296.5)
- added R30: 47R, Resistor_SMD:R_0805_2012Metric_Pad1.20x1.40mm_HandSolder, F.Cu at (-128.6, 292.5)
- added R31: 13K, Resistor_SMD:R_0805_2012Metric_Pad1.20x1.40mm_HandSolder, F.Cu at (-128.6, 297.1)
- added R32: 100K, Resistor_SMD:R_0805_2012Metric_Pad1.20x1.40mm_HandSolder, F.Cu at (-128.6, 299.2)
- added R33: 2K2, Resistor_SMD:R_0805_2012Metric_Pad1.20x1.40mm_HandSolder, F.Cu at (-154.9, 298.4)
- added R34: 2K2, Resistor_SMD:R_0805_2012Metric_Pad1.20x1.40mm_HandSolder, F.Cu at (-73.0, 286.4)
- added U11: DG611E, ThinMiniQFN:ThinMiniQFN-16_2.6mm_1.8mm, F.Cu at (232.9, 373.6)
- added U15: TPS54202DDC, Package_TO_SOT_SMD:SOT-23-6, F.Cu at (-134.0, 300.4)
- C2: renamed from C1; moved to B.Cu
- C3: renamed from C2; moved to B.Cu
- C4: renamed from C3; moved to B.Cu
- C49: value 100nF -> 100nF 20V X5R; footprint Capacitor_SMD:C_0805_2012Metric_Pad1.18x1.45mm_HandSolder -> Resistor_SMD:R_1206_3216Metric_Pad1.30x1.75mm_HandSolder
- C5: renamed from C4; moved to B.Cu
- C55: value 10uF -> 4.7uF
- C6: renamed from C5; moved to B.Cu
- C7: renamed from C6; moved to B.Cu
- D2, JP1, JP2, R1: moved to B.Cu
- JP11: renamed from JP9; moved to B.Cu
- JP12: renamed from JP10; moved to B.Cu
- JP3: renamed from JP12; moved to B.Cu
- JP4: renamed from JP11; moved to B.Cu
- JP5: renamed from JP3; moved to B.Cu
- JP6: renamed from JP4; moved to B.Cu
- JP7: renamed from JP5; moved to B.Cu
- JP8: renamed from JP6; moved to B.Cu
- R3: renamed from R2; moved to B.Cu
- RL1: footprint Relay_THT:Relay_DPDT_Omron_G2RL -> Relay_SMD:Relay_Fujitsu_FTR-B3S; moved to F.Cu
- SW2: renamed from SW1; footprint Resistor_SMD:R_0805_2012Metric_Pad1.20x1.40mm_HandSolder -> DailywellSwitches:Dailywell_SPDT
- TP1, TP2, TP3: footprint TestPoint:TestPoint_Pad_1.0x1.0mm -> TestPoint:TestPoint_Pad_D1.0mm
- U16: value SE82XX-33 -> NCV5501TG; footprint Package_TO_SOT_SMD:SOT-223-3_TabPin2 -> Package_TO_SOT_SMD:TO-252-2
- U2: renamed from U7; footprint Package_DFN_QFN:QFN-32-1EP_5x5mm_P0.5mm_EP3.45x3.45mm -> QFN-32-1EP_5x5mm_TestPoints:QFN-32-1EP_5x5mm_P0.5mm_EP3.3x3.3mm_TestPoints
- moved C49 311.2 mm to (-138.4, 299.7), turned to 90 degrees
- moved U8 291.6 mm to (367.6, 370.4)
- moved TP2 287.9 mm to (-154.9, 290.1)
- moved C25 286.5 mm to (371.5, 370.5), turned to 90 degrees
- moved C26 277.9 mm to (359.9, 369.7), turned to 180 degrees
- moved R14 277.8 mm to (359.9, 367.5), turned to 180 degrees
- moved TP1 276.5 mm to (-152.1, 304.0)
- moved C24 274.1 mm to (359.9, 371.9), turned to 180 degrees
- moved C27 272.4 mm to (355.9, 367.5), turned to 180 degrees
- moved R15 270.5 mm to (355.9, 369.7), turned to 180 degrees
- moved D4 265.7 mm to (355.9, 371.9), turned to 180 degrees
- moved C42 257.2 mm to (407.7, 126.6), turned to 180 degrees
- moved U13 256.9 mm to (401.3, 129.5)
- moved C43 254.0 mm to (394.8, 131.4)
- moved R26 253.3 mm to (407.7, 128.9), turned to 180 degrees
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- renumbered C16 to C1, C13 to C12, C14 to C13, C15 to C14, C18 to C15, C8 to C16, C20 to C17, C23 to C18, C12 to C19, C25 to C20, C26 to C21, C27 to C22, C28 to C23, C29 to C24, C30 to C25, C31 to C26, C32 to C27, C33 to C28, C34 to C29, C35 to C30, C36 to C31, C37 to C32, C38 to C33, C39 to C34, C40 to C35, C41 to C36, C43 to C37, C44 to C38, C45 to C39, C46 to C40, C47 to C41, C48 to C42, C50 to C43, C51 to C44, C52 to C45, C53 to C46, C54 to C47, C7 to C8, J2 to J3, J3 to J4, JP8 to JP10, JP7 to JP9, J1 to J_FOOTSW1, J4 to J_PWR1, R14 to R12, R15 to R13, R16 to R14, R17 to R15, R18 to R16, R19 to R17, R20 to R18, R21 to R19, R12 to R2, R22 to R20, R23 to R21, R24 to R22, R25 to R23, R26 to R24, R27 to R25, R28 to R26, R6 to R27, R29 to R28, R30 to R29, R3 to R4, R4 to R5, R5 to R6, SW5 to SW1, SW2 to SW3, U2 to U1, U12 to U10, U13 to U12, U6 to U13, U15 to U14, U1 to U5, U8 to U6, U9 to U7, U10 to U8, U11 to U9
Connections:
- C12 pad 2: -5V -> /StateVariableFilter/NegVoltRail2/NEG_VPP_OUT
- C15 pad 2: -5V -> /InputBuffer/NegVoltRail3/NEG_VPP_OUT
- C18 pad 2: -5V -> /OutputBuffer/NegVoltRail3/NEG_VPP_OUT
- C23 pad 1: -5V -> /StateVariableFilter/NegVoltRail2/NEG_VPP_OUT
- C27 pad 1: -5V -> /StateVariableFilter/NegVoltRail1/NEG_VPP_OUT
- C31 pad 1: -5V -> /InputBuffer/NegVoltRail3/NEG_VPP_OUT
- C35 pad 1: -5V -> /OutputBuffer/NegVoltRail3/NEG_VPP_OUT
- C37 pad 2: -5V -> /AnalogSwitch/NegVoltRail4/NEG_VPP_OUT
- C41 pad 1: -5V -> /AnalogSwitch/NegVoltRail4/NEG_VPP_OUT
- C43 pad 2: -5V -> /MicroController/ENV_CLK_MIX/NegVoltRail5/NEG_VPP_OUT
- C47 pad 1: -5V -> /MicroController/ENV_CLK_MIX/NegVoltRail5/NEG_VPP_OUT
- C49 pad 1: +5V -> /PSU/TPS563200_BUCK_MISC/BUCK_VIN
- C49 pad 2: -5V -> GNDS
- C55 pad 2: GND -> GNDS
- C9 pad 2: -5V -> /StateVariableFilter/NegVoltRail1/NEG_VPP_OUT
- J3 pad 6: /MicroController/SWO -> unconnected-(J3-Pad6)
- J_PWR1 pad 2: +9V -> /PSU/VIN
- R12 pad 2: -5V -> /StateVariableFilter/NegVoltRail2/NEG_VPP_OUT
- R13 pad 1: -5V -> /StateVariableFilter/NegVoltRail2/NEG_VPP_OUT
- R14 pad 2: -5V -> /StateVariableFilter/NegVoltRail1/NEG_VPP_OUT
- R15 pad 1: -5V -> /StateVariableFilter/NegVoltRail1/NEG_VPP_OUT
- R16 pad 2: -5V -> /InputBuffer/NegVoltRail3/NEG_VPP_OUT
- R17 pad 1: -5V -> /InputBuffer/NegVoltRail3/NEG_VPP_OUT
- R18 pad 2: -5V -> /OutputBuffer/NegVoltRail3/NEG_VPP_OUT
- R19 pad 1: -5V -> /OutputBuffer/NegVoltRail3/NEG_VPP_OUT
- R20 pad 2: -5V -> /AnalogSwitch/NegVoltRail4/NEG_VPP_OUT
- R21 pad 1: -5V -> /AnalogSwitch/NegVoltRail4/NEG_VPP_OUT
- R28 pad 2: -5V -> /MicroController/ENV_CLK_MIX/NegVoltRail5/NEG_VPP_OUT
- R29 pad 1: -5V -> /MicroController/ENV_CLK_MIX/NegVoltRail5/NEG_VPP_OUT
- TP1 pad 1: /MicroController/PC14 -> /PSU/TPS563200_BUCK_MISC/BUCK_VIN
- TP2 pad 1: /MicroController/PC15 -> +5V
- TP3 pad 1: /MicroController/PB0 -> +3V3
- U13 pad 4: -5V -> /MicroController/ENV_CLK_MIX/NegVoltRail5/NEG_VPP_OUT
- U16 pad 1: GND -> +5V
- U16 pad 2: +3V3 -> GNDS
- U16 pad 3: +9V -> +3V3
- U3 pad 4: -5V -> /StateVariableFilter/NegVoltRail1/NEG_VPP_OUT
- U4 pad 4: -5V -> /StateVariableFilter/NegVoltRail2/NEG_VPP_OUT
- U5 pad 4: -5V -> /InputBuffer/NegVoltRail3/NEG_VPP_OUT
- U6 pad 4: -5V -> /OutputBuffer/NegVoltRail3/NEG_VPP_OUT
Routing:
- net +5V: track 0.00 -> 134.5 mm
- net +3V3: track 0.00 -> 50.0 mm, vias 0 -> 3
- net /MicroController/NRST: track 0.00 -> 38.8 mm, vias 0 -> 2
- net /MicroController/SWDIO: track 0.00 -> 20.6 mm
- net /MicroController/SWCLK: track 0.00 -> 19.4 mm
- net Net-(C50-Pad2): track 0.00 -> 18.3 mm
- net Net-(R5-Pad2): track 0.00 -> 17.3 mm, vias 0 -> 2
- net /StateVariableFilter/NegVoltRail1/NEG_VPP_OUT: track 0.00 -> 12.2 mm
- net /InputBuffer/NegVoltRail3/NEG_VPP_OUT: track 0.00 -> 11.1 mm
- net /StateVariableFilter/NegVoltRail2/NEG_VPP_OUT: track 0.00 -> 10.8 mm
- net /MicroController/BOOT0: track 0.00 -> 10.5 mm, vias 0 -> 1
- net /OutputBuffer/NegVoltRail3/NEG_VPP_OUT: track 0.00 -> 10.2 mm
- net Net-(C19-Pad1): track 0.00 -> 9.88 mm, vias 0 -> 1
- net Net-(C51-Pad1): track 0.00 -> 9.34 mm
- net /PSU/TPS563200_BUCK_MISC/BUCK_VIN: track 0.00 -> 9.17 mm
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